Commit message: :truck: change package name

File: snapbot/snapbot_description/urdf/ur3e.urdf (robot description, URDF)
Before this commit: robot ur3e, 21 links, 20 joints
Links:
- link camera_link: geometry collision box size=0.02505 0.025 0.09; visual mesh filename=package://snapbot_description/meshes/sensors/d435.STL
- link display: geometry collision box size=0.2665 0.179 0.0615; visual mesh filename=package://snapbot_description/meshes/ur3e/visual/display.stl scale=0.001 0.001 0.001
- link ur3ebase_link_inertia: geometry collision mesh filename=package://snapbot_description/meshes/ur3e/collision/base.stl; visual mesh filename=package://snapbot_description/meshes/ur3e/visual/base.dae
- link ur3eforearm_link: geometry collision mesh filename=package://snapbot_description/meshes/ur3e/collision/forearm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; visual mesh filename=package://snapbot_description/meshes/ur3e/visual/forearm.dae
- link ur3eshoulder_link: geometry collision mesh filename=package://snapbot_description/meshes/ur3e/collision/shoulde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; visual mesh filename=package://snapbot_description/meshes/ur3e/visual/shoulder.d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
- link ur3eupper_arm_link: geometry collision mesh filename=package://snapbot_description/meshes/ur3e/collision/upperar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; visual mesh filename=package://snapbot_description/meshes/ur3e/visual/upperarm.d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
- link ur3ewrist_1_link: geometry collision mesh filename=package://snapbot_description/meshes/ur3e/collision/wrist1.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; visual mesh filename=package://snapbot_description/meshes/ur3e/visual/wrist1.dae
- link ur3ewrist_2_link: geometry collision mesh filename=package://snapbot_description/meshes/ur3e/collision/wrist2.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; visual mesh filename=package://snapbot_description/meshes/ur3e/visual/wrist2.dae
- link ur3ewrist_3_link: geometry collision mesh filename=package://snapbot_description/meshes/ur3e/collision/wrist3.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; visual mesh filename=package://snapbot_description/meshes/ur3e/visual/wrist3.dae
